Commit message: turtlebot settings changes

File: turtlebot3_description/urdf/turtlebot3_burger_marker.gazebo.xacro (robot description, xacro)
@@ -48,5 +48,5 @@
       <odometryFrame>odom</odometryFrame>
       <odometrySource>world</odometrySource>
-      <publishOdomTF>false</publishOdomTF>
+      <publishOdomTF>true</publishOdomTF>
       <robotBaseFrame>base_footprint</robotBaseFrame>
       <publishWheelTF>false</publishWheelTF>

File: turtlebot3_description/urdf/turtlebot3_burger_marker.urdf.xacro (robot description, xacro)
@@ -4,7 +4,4 @@
   <xacro:include filename="$(find turtlebot3_description)/urdf/turtlebot3_burger.gazebo.xacro"/>
   <link name="base_footprint"/>
-  <visual>
-      <origin xyz="0 0 0.0" rpy="0 0 1.57"/>
-    </visual>
   <joint name="base_joint" type="fixed">
     <parent link="base_footprint"/>
@@ -33,6 +30,5 @@
                izz="2.0064271e-03" />
     </inertial>
-  </link>
- <link name="aruco_marker_2">
+  <link name="aruco_marker_2">
     <visual>
       <origin xyz="0 0 0" rpy="0 0 0"/>
@@ -61,4 +57,5 @@
     <origin xyz="-0.03 0 0.19" rpy="0 -1.57 0"/>
   </joint>
+  </link>
   <joint name="wheel_left_joint" type="continuous">
     <parent link="base_link"/>
